Commit message: Weed now works

File: urdf/gripper.urdf (robot description, URDF)
Before this commit: robot gripper, 4 links, 3 joints
Links:
- removed link end_effector_left
- removed link left_tool
- removed link leftgripper2_link
- removed link leftgripper_link
- added link red_end_effector_left; collision mesh filename=package://hdt_michigan_description/meshes/PINCER_HOUSING2.S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; visual mesh filename=package://hdt_michigan_description/meshes/PINCER_HOUSING2.S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
- added link red_left_tool; visual sphere radius=0.002
- added link red_leftgripper2_link; collision mesh filename=package://hdt_michigan_description/meshes/PINCER_FINGER.STL; visual mesh filename=package://hdt_michigan_description/meshes/PINCER_FINGER.STL
- added link red_leftgripper_link; collision mesh filename=package://hdt_michigan_description/meshes/PINCER_FINGER.STL; visual mesh filename=package://hdt_michigan_description/meshes/PINCER_FINGER.STL
Joints:
- removed joint left_tool_joint
- removed joint leftgripper
- removed joint leftgripper2
- added joint red_left_tool_joint: type fixed, parent red_end_effector_left, child red_left_tool, origin xyz=0.0 0.0 0.181 rpy=0 0 0
- added joint red_leftgripper: type fixed, parent red_end_effector_left, child red_leftgripper_link, origin xyz=0 0.0135 0.068553 rpy=1.5707 -0.42 -1.5707, axis 0 0 1
- added joint red_leftgripper2: type fixed, parent red_end_effector_left, child red_leftgripper2_link, origin xyz=0 -0.0135 0.068553 rpy=1.5707 -0.42 1.5707, axis 0 0 1
